File: hw/heliosphere.kicad_pcb (KiCad board)
At the start: 2 copper layers, 250 x 50 mm, 16 parts, among them J101 Conn_01x02

Commit message: footprint and schematic update
Parts:
- added J102: Conn_01x02, Connector_Wire:SolderWire-2.5sqmm_1x02_P8.8mm_D2.4mm_OD4.4mm, F.Cu at (25.7, 61.5)
- D101, D102, D103, D104, D105: moved to B.Cu
- moved R101 239.6 mm to (25.5, 45.3)
- moved J101 239.3 mm to (25.7, 56.1), turned to 0 degrees
- moved D106 239.2 mm to (25.9, 30.8)
- moved REF** 234.7 mm to (258.0, 30.5)
- moved REF** 230.6 mm to (254.8, 23.5)
- moved D101 205.2 mm to (42.5, 37.5), turned to 0 degrees
- moved D105 200.2 mm to (242.5, 37.5), turned to 0 degrees
- moved REF** 173.1 mm to (254.5, 59.0)
- moved RV105 156.0 mm to (217.5, 42.5)
- moved RV101 153.2 mm to (62.9, 42.5)
- moved RV102 135.0 mm to (72.0, 42.5)
- moved D102 107.7 mm to (92.5, 37.5), turned to 0 degrees
- moved D104 102.9 mm to (192.5, 37.5), turned to 0 degrees
- moved RV104 56.0 mm to (167.5, 42.5)
- moved RV103 44.0 mm to (117.5, 42.5)
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Routing:
- net Net-(D106-K): track 262.7 -> 226.5 mm
- net Net-(J101-Pin_1): track 8.49 -> 13.4 mm
- net Net-(D105-A): track 24.7 -> 29.0 mm
- net Net-(D104-A): track 24.7 -> 29.0 mm
- net Net-(D103-A): track 24.7 -> 29.0 mm
- net Net-(D102-A): track 20.3 -> 24.5 mm
- net Net-(D101-A): track 27.5 -> 30.4 mm
- net GND: vias 54 -> 4
Other:
- board size 250 x 50 mm -> 240 x 45 mm
- board text added: "10mm spacing"
- board text added: "50x50 mm spacing"
- board text added: "5mm spacing"
- board text added: "PCB FACE UP"
- board text added: "SOLDER LEDS FACE DOWN ON BACKSIDE"
- board text removed: "SOLDER LEDS FACE DOWN"

Commit message: swap trimpot for available one on mouser
Parts:
- removed RV101, RV102, RV103, RV104, RV105: 20, footprints:dale_1680_trimpot
- added VR101: 3266W-1-200LF, footprints:bourns3266W_1_200LF, F.Cu at (62.0, 45.3)
- added VR102: 3266W-1-200LF, footprints:bourns3266W_1_200LF, F.Cu at (70.5, 45.3)
- added VR103: 3266W-1-200LF, footprints:bourns3266W_1_200LF, F.Cu at (116.3, 45.3)
- added VR104: 3266W-1-200LF, footprints:bourns3266W_1_200LF, F.Cu at (166.3, 45.3)
- added VR105: 3266W-1-200LF, footprints:bourns3266W_1_200LF, F.Cu at (216.3, 45.3)
Routing:
- net Net-(D106-K): track 226.5 -> 271.6 mm
- net Net-(D102-A): track 24.5 -> 28.8 mm
- net Net-(D103-A): track 29.0 -> 33.0 mm
- net Net-(D105-A): track 29.0 -> 33.0 mm
- net Net-(D104-A): track 29.0 -> 33.0 mm
- net Net-(D101-A): track 30.4 -> 32.3 mm
Other:
- board text removed: "CW Ω↑ CCW Ω↓"
